Commit message: fix tf publisher, include static transform in launch file, change robot model urdf

File: bluerov_model/BlueRov2.urdf.xacro (robot description, xacro)
@@ -119,5 +119,5 @@
     </buoyancy>
   </link>
-  <link name="dvl_link">
+  <!-- <link name="dvl_link">
   </link>
   <joint name="dvl_joint" type="fixed">
@@ -125,5 +125,5 @@
     <child link="dvl_link"/>
     <origin xyz="0.042 -0.08904 -0.21062" rpy="3.141592653589793 0 -1.5707963267948966"/>
-  </joint>
+  </joint> -->
   <link name="camera_link">
     <!-- visual>
